File: cad_files/Real_time_clock.kicad_pcb (KiCad board)
At the start: 2 copper layers, 49 x 65 mm, 36 parts, among them J1 USB_C_Receptacle_USB2.0, J2 RJ11, J3 RJ11, J4 PH, J5 PH, J6 Conn_02x03_Odd_Even, SW1 SW_Push, U1 SY8401ABC, U2 AMS1117-3.3, U3 EDGE_STM32F405_CPU_V1

Commit message: ready for fab
Parts:
- added BT1: Battery_Cell, Evezor_extras:BatteryHolder_Keystone_1060_1x2032, F.Cu at (128.7, 104.8)
- added C11: 1F, Capacitor_THT:CP_Radial_D8.0mm_P3.50mm, F.Cu at (132.0, 90.5)
- added C12: 12.5pF, Capacitor_SMD:C_0603_1608Metric, F.Cu at (114.8, 92.4)
- added C13: .1uF, Capacitor_SMD:C_0603_1608Metric, F.Cu at (126.5, 87.0)
- added C7: 12.5pF, Capacitor_SMD:C_0603_1608Metric, F.Cu at (114.8, 85.5)
- added D7: 1n4148, Diode_SMD:D_SOD-123, F.Cu at (138.5, 92.8)
- added D8: 1n4148, Diode_SMD:D_SOD-123, F.Cu at (138.5, 87.0)
- added D9: LED, LED_SMD:LED_0603_1608Metric, F.Cu at (120.1, 84.4)
- added R6: 4.7k, Resistor_SMD:R_0603_1608Metric, F.Cu at (137.2, 118.0)
- added R7: 4.7k, Resistor_SMD:R_0603_1608Metric, F.Cu at (137.2, 116.0)
- added R8: 15k, Resistor_SMD:R_0603_1608Metric, F.Cu at (122.1, 84.5)
- added SW2: SW_Push, EvezorLIB:SWITCH_2x3_SMD_TACTILE_GREEN, F.Cu at (113.6, 119.3)
- added SW3: SW_Push, EvezorLIB:SWITCH_2x3_SMD_TACTILE_GREEN, F.Cu at (122.6, 119.3)
- added U4: RTC_REAL_TIME_CLOCK_PCF8563, Package_SO:SOIC-8_3.9x4.9mm_P1.27mm, F.Cu at (121.0, 90.1)
- added Y1: Crystal, EvezorLIB:CRYSTAL_SEIKO_32.768_SC-32S32.768kHz20PPM12.5pF, F.Cu at (114.3, 88.8)
- moved G*** 16.8 mm to (111.3, 91.7), turned to 90 degrees
- moved REF** 7.68 mm to (112.1, 111.1)
- moved G*** 6.48 mm to (111.3, 99.0), turned to 90 degrees
Connections:
- U3 pad 12: Net-(U3-Pad12) -> /SCL
- U3 pad 13: Net-(U3-Pad13) -> /SDA
- U3 pad 30: Net-(U3-Pad30) -> /BUTTON_B
- U3 pad 31: Net-(U3-Pad31) -> /BUTTON_A
Routing:
- net /SDA: track 0.00 -> 37.8 mm, vias 0 -> 2
- net /SCL: track 0.00 -> 34.4 mm, vias 0 -> 2
- net +3V3: track 107.4 -> 135.0 mm, vias 4 -> 3
- net /CLKPWR: track 0.00 -> 19.1 mm
- net Net-(BT1-Pad1): track 0.00 -> 13.3 mm
- net /BUTTON_B: track 0.00 -> 9.18 mm, vias 0 -> 1
- net /OSCO: track 0.00 -> 6.94 mm
- net /OSCI: track 0.00 -> 6.72 mm
- net /CLKOUT: track 0.00 -> 6.54 mm
- net /BUTTON_A: track 0.00 -> 5.06 mm, vias 0 -> 1
- net GND: track 18.9 -> 21.6 mm, vias 93 -> 143
- net Net-(D9-Pad1): track 0.00 -> 2.03 mm
- net /OLED_SCL: track 10.1 -> 8.49 mm
- net /RESET: track 14.0 -> 14.6 mm
Other:
- board size 49 x 65 mm -> 49 x 70 mm
- board text added: "A"
- board text added: "B"
- board text added: "REAL TIME CLOCK V1.0p"
- board text removed: "THE THING V1.0P"
- board text removed: "www.evezor.com/products/thisProduct"
